Commit message: Updated workspace

File: chapter_3_ws/src/robot_description/urdf/gazebo_essentials.xacro (robot description, xacro)
@@ -1,2 +1,3 @@
+<<<<<<< HEAD
 <?xml version="1.0"?>
 <robot xmlns:xacro="http://ros.org/wiki/xacro" name="gazebo_essentials" >
@@ -50,2 +51,55 @@
 <!--######################################################################-->
 </robot>
+=======
+<?xml version="1.0"?>
+<robot xmlns:xacro="http://ros.org/wiki/xacro" name="gazebo_essentials" >
+<!--############################# ROS-CONTROL #########################################-->
+<gazebo>
+    <plugin name="gazebo_ros_control" filename="libgazebo_ros_control.so">
+      <robotNamespace>/</robotNamespace>
+      <controlPeriod>0.001</controlPeriod>
+      <legacyModeNS>false</legacyModeNS>
+    </plugin>
+  </gazebo>
+<!--################################ ROS-Controllers ######################################-->
+<gazebo>
+      <plugin name="diff_drive_controller" filename="libgazebo_ros_diff_drive.so">
+        <legacyMode>false</legacyMode>
+        <alwaysOn>true</alwaysOn>
+        <updateRate>1000.0</updateRate>
+        <leftJoint>front_left_wheel_joint, rear_left_wheel_joint</leftJoint>
+        <rightJoint>front_right_wheel_joint, rear_right_wheel_joint</rightJoint>
+        <wheelSeparation>0.5</wheelSeparation>
+        <wheelDiameter>0.2</wheelDiameter>
+        <wheelTorque>10</wheelTorque>
+        <publishTf>1</publishTf>
+        <odometryFrame>map</odometryFrame>
+        <commandTopic>cmd_vel</commandTopic>
+        <odometryTopic>odom</odometryTopic>
+        <robotBaseFrame>base_link</robotBaseFrame>
+        <wheelAcceleration>2.8</wheelAcceleration>
+        <publishWheelJointState>true</publishWheelJointState>
+        <publishWheelTF>false</publishWheelTF>
+        <odometrySource>world</odometrySource>
+        <rosDebugLevel>Debug</rosDebugLevel>
+      </plugin>
+</gazebo>
+<!--######################################################################-->
+  <gazebo>
+    <plugin name="joint_state_publisher" filename="libgazebo_ros_joint_state_publisher.so">
+      <jointName>arm_base_joint, shoulder_joint, bottom_wrist_joint, elbow_joint, bottom_wrist_joint</jointName>
+    </plugin>
+  </gazebo>
+<!--############################# Wheel friction #########################################-->
+<xacro:macro name="wheel_friction" params="prefix ">
+<gazebo reference="${prefix}_wheel">
+ <mu1 value="1.0"/>
+ <mu2 value="1.0"/>
+ <kp value="10000000.0" />
+ <kd value="1.0" />
+ <fdir1 value="1 0 0"/>
+</gazebo>
+</xacro:macro>
+<!--######################################################################-->
+</robot>
+>>>>>>> adding all codes

File: chapter_3_ws/src/robot_description/urdf/mobile_manipulator.urdf.xacro (robot description, xacro)
@@ -1,2 +1,3 @@
+<<<<<<< HEAD
 <?xml version="1.0"?>
 <robot xmlns:xacro="http://ros.org/wiki/xacro" name="robot_base" >
@@ -5,2 +6,10 @@
 <xacro:arm_joint prefix="arm_base_link" parent="base_link" child="arm_base" originxyz="0.20 0.0 0.145" originrpy="0 0 0"/>
 </robot>
+=======
+<?xml version="1.0"?>
+<robot xmlns:xacro="http://ros.org/wiki/xacro" name="robot_base" >
+<xacro:include filename="$(find robot_description)/urdf/robot_base.urdf.xacro" />
+<xacro:include filename="$(find robot_description)/urdf/robot_arm.urdf.xacro" />
+<xacro:arm_joint prefix="arm_base_link" parent="base_link" child="arm_base" originxyz="0.20 0.0 0.145" originrpy="0 0 0"/>
+</robot>
+>>>>>>> adding all codes

File: chapter_3_ws/src/robot_description/urdf/robot_base.urdf.xacro (robot description, xacro)
@@ -1,2 +1,3 @@
+<<<<<<< HEAD
 <?xml version="1.0"?>
 <robot xmlns:xacro="http://ros.org/wiki/xacro" name="robot_base" >
@@ -63,2 +64,68 @@
 <!--#####################################################################################-->
 </robot>
+=======
+<?xml version="1.0"?>
+<robot xmlns:xacro="http://ros.org/wiki/xacro" name="robot_base" >
+<xacro:include filename="$(find robot_description)/urdf/robot_essentials.xacro" />
+<xacro:include filename="$(find robot_description)/urdf/gazebo_essentials.xacro" />
+<!--######################################################################-->
+  <link name="base_link">
+    <inertial>
+      <origin
+        xyz="0.0030946 4.78250032638821E-11 0.053305"
+        rpy="0 0 0" />
+      <mass
+        value="47.873" />
+      <inertia
+        ixx="0.774276574699151"
+        ixy="-1.03781944357671E-10"
+        ixz="0.00763014265820928"
+        iyy="1.64933255189991"
+        iyz="1.09578155845563E-12"
+        izz="2.1239326987473" />
+    </inertial>
+    <visual>
+      <origin
+        xyz="0 0 0"
+        rpy="1.5707963267949 0 3.14" />
+      <geometry>
+        <mesh filename="package://robot_description/meshes/robot_base.stl" />
+      </geometry>
+      <material
+        name="">
+        <color
+          rgba="0.79216 0.81961 0.93333 1" />
+      </material>
+    </visual>
+    <collision>
+      <origin
+        xyz="0 0 0"
+        rpy="1.5707963267949 0 3.14" />
+      <geometry>
+        <mesh filename="package://robot_description/meshes/robot_base.stl" />
+      </geometry>
+    </collision>
+  </link>
+<!--############################# Remaining wheels #########################################-->
+<xacro:robot_wheel prefix="front_left"/>
+<xacro:robot_wheel prefix="front_right"/>
+<xacro:robot_wheel prefix="rear_left"/>
+<xacro:robot_wheel prefix="rear_right"/>
+<!--############################# Wheel Joints #########################################-->
+<xacro:wheel_joint prefix="front_left" origin="0.220 0.250 0"/>
+<xacro:wheel_joint prefix="front_right" origin="0.220 -0.250 0"/>
+<xacro:wheel_joint prefix="rear_left" origin="-0.220 0.250 0"/>
+<xacro:wheel_joint prefix="rear_right" origin="-0.220 -0.250 0"/>
+<!--############################# Wheel Transmissions #########################################-->
+<xacro:base_transmission prefix="front_left"/>
+<xacro:base_transmission prefix="front_right"/>
+<xacro:base_transmission prefix="rear_left"/>
+<xacro:base_transmission prefix="rear_right"/>
+<!--############################# Wheel Friction #########################################-->
+<xacro:wheel_friction prefix="front_left"/>
+<xacro:wheel_friction prefix="front_right"/>
+<xacro:wheel_friction prefix="rear_left"/>
+<xacro:wheel_friction prefix="rear_right"/>
+<!--#####################################################################################-->
+</robot>
+>>>>>>> adding all codes

File: chapter_3_ws/src/robot_description/urdf/robot_essentials.xacro (robot description, xacro)
@@ -1,2 +1,3 @@
+<<<<<<< HEAD
 <?xml version="1.0"?>
 <robot xmlns:xacro="http://ros.org/wiki/xacro" name="robot_essentials" >
@@ -85,2 +86,90 @@
 <!--######################################################################-->
 </robot>
+=======
+<?xml version="1.0"?>
+<robot xmlns:xacro="http://ros.org/wiki/xacro" name="robot_essentials" >
+<!--######################################################################-->
+<xacro:macro name="robot_wheel" params="prefix">
+<link name="${prefix}_wheel">
+    <inertial>
+      <origin
+        xyz="-4.1867E-18 0.0068085 -1.65658661799998E-18"
+        rpy="0 0 0" />
+      <mass
+        value="2.6578" />
+      <inertia
+        ixx="0.00856502765719703"
+        ixy="1.5074118157338E-19"
+        ixz="-4.78150098725052E-19"
+        iyy="0.013670640432096"
+        iyz="-2.68136447099727E-19"
+        izz="0.00856502765719703" />
+    </inertial>
+    <visual>
+      <origin
+        xyz="0 0 0"
+        rpy="1.5707963267949 0 0" />
+      <geometry>
+        <mesh filename="package://robot_description/meshes/wheel.stl" />
+      </geometry>
+      <material
+        name="">
+        <color
+          rgba="0.79216 0.81961 0.93333 1" />
+      </material>
+    </visual>
+    <collision>
+      <origin
+        xyz="0 0 0"
+        rpy="1.5707963267949 0 0" />
+      <geometry>
+        <mesh filename="package://robot_description/meshes/wheel.stl" />
+      </geometry>
+    </collision>
+  </link>
+</xacro:macro>
+<!--######################################################################-->
+<xacro:macro name="wheel_joint" params="prefix origin">
+<joint name="${prefix}_wheel_joint" type="continuous">
+    <axis xyz="0 1 0"/>
+    <parent link ="base_link"/>
+    <child link ="${prefix}_wheel"/>
+    <origin rpy ="0 0 0" xyz= "${origin}"/>
+  </joint>
+</xacro:macro>
+<xacro:macro name="arm_joint" params="prefix parent child originxyz originrpy">
+<joint name="${prefix}_joint" type="continuous">
+  <axis xyz="0 0 1"/>
+  <parent link="${parent}"/>
+  <child link="${child}"/>
+  <origin rpy="${originrpy}" xyz="${originxyz}"/>
+</joint>
+</xacro:macro>
+<!--######################################################################-->
+<xacro:macro name="base_transmission" params="prefix ">
+<transmission name="${prefix}_wheel_trans" type="SimpleTransmission">
+  <type>transmission_interface/SimpleTransmission</type>
+  <actuator name="${prefix}_wheel_motor">
+   <hardwareInterface>hardware_interface/VelocityJointInterface</hardwareInterface>
+   <mechanicalReduction>1</mechanicalReduction>
+  </actuator>
+  <joint name="${prefix}_wheel_joint">
+   <hardwareInterface>hardware_interface/VelocityJointInterface</hardwareInterface>
+  </joint>
+</transmission>
+</xacro:macro>
+<xacro:macro name="arm_transmission" params="prefix ">
+<transmission name="${prefix}_trans" type="SimpleTransmission">
+  <type>transmission_interface/SimpleTransmission</type>
+  <actuator name="${prefix}_motor">
+   <hardwareInterface>hardware_interface/PositionJointInterface</hardwareInterface>
+   <mechanicalReduction>1</mechanicalReduction>
+  </actuator>
+  <joint name="${prefix}_joint">
+   <hardwareInterface>hardware_interface/PositionJointInterface</hardwareInterface>
+  </joint>
+</transmission>
+</xacro:macro>
+<!--######################################################################-->
+</robot>
+>>>>>>> adding all codes
